File: KiCAD/Amplifier_x8.kicad_sch (KiCad schematic)
At the start: 28 parts, among them U4 AD8534ARZ-REEL, U5 AD8534ARZ-REEL

Commit message: Finished routing
Connections:
- net IN2: now also U4.12 (+); no longer U4.5 (+)
- net IN4: now also U4.5 (+); no longer U4.12 (+)
- net IN6: now also U5.12 (+); no longer U5.5 (+)
- net IN8: now also U5.5 (+); no longer U5.12 (+)
- net OUT1: now also R14.2, U5.8; no longer R4.2, U4.1
- net OUT2: now also R13.2, U5.7; no longer R5.2, U4.7
- net OUT3: now also R12.2, U5.1; no longer R6.2, U4.8
- net OUT4: now also R15.2, U5.14; no longer R7.2, U4.14
- net OUT5: now also R6.2, U4.8; no longer R12.2, U5.1
- net OUT6: now also R5.2, U4.7; no longer R13.2, U5.7
- net OUT7: now also R4.2, U4.1; no longer R14.2, U5.8
- net OUT8: now also R7.2, U4.14; no longer R15.2, U5.14
Changed lines of the file:
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@@
 	(hierarchical_label "OUT3"
 		(shape output)
-		(at 195.58 63.5 0)
+		(at 73.66 121.92 0)
 		(effects
 			(font
@@
 	(hierarchical_label "OUT2"
 		(shape output)
-		(at 134.62 63.5 0)
+		(at 134.62 121.92 0)
 		(effects
 			(font
@@
 	(hierarchical_label "OUT7"
 		(shape output)
-		(at 195.58 121.92 0)
+		(at 73.66 63.5 0)
 		(effects
 			(font
@@
 	(hierarchical_label "IN6"
 		(shape input)
-		(at 106.68 124.46 180)
+		(at 228.6 124.46 180)
 		(effects
 			(font
@@
 	(hierarchical_label "IN8"
 		(shape input)
-		(at 228.6 124.46 180)
+		(at 106.68 124.46 180)
 		(effects
 			(font
@@
 	(hierarchical_label "OUT4"
 		(shape output)
-		(at 256.54 63.5 0)
+		(at 256.54 121.92 0)
 		(effects
 			(font
@@
 	(hierarchical_label "OUT8"
 		(shape output)
-		(at 256.54 121.92 0)
+		(at 256.54 63.5 0)
 		(effects
 			(font
@@
 	(hierarchical_label "IN2"
 		(shape input)
-		(at 106.68 66.04 180)
+		(at 228.6 66.04 180)
 		(effects
 			(font
@@
 	(hierarchical_label "OUT5"
 		(shape output)
-		(at 73.66 121.92 0)
+		(at 195.58 63.5 0)
 		(effects
 			(font
@@
 	(hierarchical_label "OUT1"
 		(shape output)
-		(at 73.66 63.5 0)
+		(at 195.58 121.92 0)
 		(effects
 			(font
@@
 	(hierarchical_label "IN4"
 		(shape input)
-		(at 228.6 66.04 180)
+		(at 106.68 66.04 180)
 		(effects
 			(font
@@
 	(hierarchical_label "OUT6"
 		(shape output)
-		(at 134.62 121.92 0)
+		(at 134.62 63.5 0)
 		(effects
 			(font

Commit message: Added a debug header
Connections:
- net IN1: now also U5.10 (+); no longer U4.3 (+)
- net IN2: now also U5.5 (+); no longer U4.12 (+)
- net IN3: now also U5.3 (+); no longer U4.10 (+)
- net IN4: now also U5.12 (+); no longer U4.5 (+)
- net IN5: now also U4.10 (+); no longer U5.3 (+)
- net IN6: now also U4.5 (+); no longer U5.12 (+)
- net IN7: now also U4.3 (+); no longer U5.10 (+)
- net IN8: now also U4.12 (+); no longer U5.5 (+)

Commit message: Added test-points
Parts:
- added TP6, TP8: Keystone_5014_Yellow, TestPoint:TestPoint_Keystone_5010-5014_Multipurpose, symbol Connectors:Keystone_5014_Yellow
Connections:
- net OUT1: now also TP8.1
- net OUT8: now also TP6.1

Commit message: Added PA_Enable pull-down and moved the debug header
Parts:
- renumbered R9 to R10, R10 to R11, R11 to R12, R12 to R13, R13 to R14, R14 to R15, R15 to R16, R16 to R17, R17 to R18, R18 to R19, R19 to R20, R4 to R5, R5 to R6, R6 to R7, R7 to R8, R8 to R9, TP6 to TP4, TP8 to TP5

Commit message: Moved the microphone RL to per-channel instead of per-mic
Parts:
- renumbered C34 to C31, C35 to C32, C36 to C33, C37 to C34, C38 to C35, C39 to C36, C40 to C37, C41 to C38, C42 to C39, C43 to C40, R13 to R10, R14 to R11, R15 to R12, R16 to R13, R17 to R14, R18 to R15, R19 to R16, R20 to R17, R5 to R2, R6 to R3, R7 to R4, R8 to R5, R9 to R6, R10 to R7, R11 to R8, R12 to R9, U4 to U3, U5 to U4

Commit message: Added title block and version text
Parts:
- renumbered C31 to C55, C32 to C56, C33 to C57, C34 to C58, C35 to C59, C36 to C60, C37 to C61, C38 to C62, C39 to C63, C40 to C64, R2 to R70, R3 to R71, R4 to R72, R5 to R73, R6 to R74, R7 to R75, R8 to R76, R9 to R77, R10 to R78, R11 to R79, R12 to R80, R13 to R81, R14 to R82, R15 to R83, R16 to R84, R17 to R85, TP4 to TP6, TP5 to TP7, U3 to U4, U4 to U5
Other:
- company: (none) -> University of Cape Town
- title: (none) -> Amplifier
