File: KiCAD/Amplifier_x8.kicad_sch (KiCad schematic)
At the start: 30 parts, among them U4 AD8534ARZ-REEL, U5 AD8534ARZ-REEL

Commit message: Final Updates:
- Mounting holes for an isolation shield
- 5V test-point to inject power
- Test signal input with resistor ladder
Parts:
- renumbered R83 to R100, R84 to R101, R85 to R102, R70 to R87, R71 to R88, R72 to R89, R73 to R90, R74 to R91, R75 to R92, R76 to R93, R77 to R94, R78 to R95, R79 to R96, R80 to R97, R81 to R98, R82 to R99, TP6 to TP8, TP7 to TP9

Commit message: Changed 100pF and 100nF to AVX parts, and gave TPA6211 a pin-1 dot
Parts:
- C55, C56, C57, C58, C59, C60, C61, C62, C63, C64: MPN GCG188R91H104KA01D -> 06035C104KAT2A; Manufacturer Murata -> KYOCERA AVX; SPN 81-GCG188R91H104KA1D -> 581-06035C104KAT2A
Changed lines of the file:
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@@
 			)
 		)
-		(property "Manufacturer" "Murata"
+		(property "Manufacturer" "KYOCERA AVX"
 			(at 165.1 62.865 0)
 			(hide yes)
@@
 			)
 		)
-		(property "MPN" "GCG188R91H104KA01D "
+		(property "MPN" "06035C104KAT2A"
 			(at 165.1 64.77 0)
 			(hide yes)
@@
 			)
 		)
-		(property "SPN" "81-GCG188R91H104KA1D "
+		(property "SPN" "581-06035C104KAT2A"
 			(at 165.1 68.58 0)
 			(hide yes)
@@
 			)
 		)
-		(property "Manufacturer" "Murata"
+		(property "Manufacturer" "KYOCERA AVX"
 			(at 165.1 121.285 0)
 			(hide yes)
@@
 			)
 		)
-		(property "MPN" "GCG188R91H104KA01D "
+		(property "MPN" "06035C104KAT2A"
 			(at 165.1 123.19 0)
 			(hide yes)
@@
 			)
 		)
-		(property "SPN" "81-GCG188R91H104KA1D "
+		(property "SPN" "581-06035C104KAT2A"
 			(at 165.1 127 0)
 			(hide yes)
@@
 			)
 		)
-		(property "Manufacturer" "Murata"
+		(property "Manufacturer" "KYOCERA AVX"
 			(at 226.06 121.285 0)
 			(hide yes)
@@
 			)
 		)
-		(property "MPN" "GCG188R91H104KA01D "
+		(property "MPN" "06035C104KAT2A"
 			(at 226.06 123.19 0)
 			(hide yes)
@@
 			)
 		)
-		(property "SPN" "81-GCG188R91H104KA1D "
+		(property "SPN" "581-06035C104KAT2A"
 			(at 226.06 127 0)
 			(hide yes)
@@
 			)
 		)
-		(property "Manufacturer" "Murata"
+		(property "Manufacturer" "KYOCERA AVX"
 			(at 104.14 62.865 0)
 			(hide yes)
@@
 			)
 		)
-		(property "MPN" "GCG188R91H104KA01D "
+		(property "MPN" "06035C104KAT2A"
 			(at 104.14 64.77 0)
 			(hide yes)
@@
 			)
 		)
-		(property "SPN" "81-GCG188R91H104KA1D "
+		(property "SPN" "581-06035C104KAT2A"
 			(at 104.14 68.58 0)
 			(hide yes)
@@
 			)
 		)
-		(property "Manufacturer" "Murata"
+		(property "Manufacturer" "KYOCERA AVX"
 			(at 55.88 159.385 0)
 			(hide yes)
@@
 			)
 		)
-		(property "MPN" "GCG188R91H104KA01D "
+		(property "MPN" "06035C104KAT2A"
 			(at 55.88 161.29 0)
 			(hide yes)
@@
 			)
 		)
-		(property "SPN" "81-GCG188R91H104KA1D "
+		(property "SPN" "581-06035C104KAT2A"
 			(at 55.88 165.1 0)
 			(hide yes)
@@
 			)
 		)
-		(property "Manufacturer" "Murata"
+		(property "Manufacturer" "KYOCERA AVX"
 			(at 43.18 159.385 0)
 			(hide yes)
@@
 			)
 		)
-		(property "MPN" "GCG188R91H104KA01D "
+		(property "MPN" "06035C104KAT2A"
 			(at 43.18 161.29 0)
 			(hide yes)
@@
 			)
 		)
-		(property "SPN" "81-GCG188R91H104KA1D "
+		(property "SPN" "581-06035C104KAT2A"
 			(at 43.18 165.1 0)
 			(hide yes)
@@
 			)
 		)
-		(property "Manufacturer" "Murata"
+		(property "Manufacturer" "KYOCERA AVX"
 			(at 43.18 62.865 0)
 			(hide yes)
@@
 			)
 		)
-		(property "MPN" "GCG188R91H104KA01D "
+		(property "MPN" "06035C104KAT2A"
 			(at 43.18 64.77 0)
 			(hide yes)
@@
 			)
 		)
-		(property "SPN" "81-GCG188R91H104KA1D "
+		(property "SPN" "581-06035C104KAT2A"
 			(at 43.18 68.58 0)
 			(hide yes)
@@
 			)
 		)
-		(property "Manufacturer" "Murata"
+		(property "Manufacturer" "KYOCERA AVX"
 			(at 104.14 121.285 0)
 			(hide yes)
@@
 			)
 		)
-		(property "MPN" "GCG188R91H104KA01D "
+		(property "MPN" "06035C104KAT2A"
 			(at 104.14 123.19 0)
 			(hide yes)
@@
 			)
 		)
-		(property "SPN" "81-GCG188R91H104KA1D "
+		(property "SPN" "581-06035C104KAT2A"
 			(at 104.14 127 0)
 			(hide yes)
@@
 			)
 		)
-		(property "Manufacturer" "Murata"
+		(property "Manufacturer" "KYOCERA AVX"
 			(at 43.18 121.285 0)
 			(hide yes)
@@
 			)
 		)
-		(property "MPN" "GCG188R91H104KA01D "
+		(property "MPN" "06035C104KAT2A"
 			(at 43.18 123.19 0)
 			(hide yes)
@@
 			)
 		)
-		(property "SPN" "81-GCG188R91H104KA1D "
+		(property "SPN" "581-06035C104KAT2A"
 			(at 43.18 127 0)
 			(hide yes)
@@
 			)
 		)
-		(property "Manufacturer" "Murata"
+		(property "Manufacturer" "KYOCERA AVX"
 			(at 226.06 62.865 0)
 			(hide yes)
@@
 			)
 		)
-		(property "MPN" "GCG188R91H104KA01D "
+		(property "MPN" "06035C104KAT2A"
 			(at 226.06 64.77 0)
 			(hide yes)
@@
 			)
 		)
-		(property "SPN" "81-GCG188R91H104KA1D "
+		(property "SPN" "581-06035C104KAT2A"
 			(at 226.06 68.58 0)
 			(hide yes)
