File: KiCAD/Sonar.kicad_sch (KiCad schematic)
At the start: 13 parts

Commit message: Regenerated CAM output
Other:
- sheet ADC ports: added nCS1, nCS2; removed CS1, CS2
- sheet Control_Power ports: added ADC1_nCS, ADC2_nCS; removed ADC1_CS, ADC2_CS
Changed lines of the file:
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@@
 		(rev "v1.0")
 		(company "University of Cape Town")
+		(comment 1 "Radar Remote Sensing Group")
+		(comment 2 "Radar Masters")
 	)
 	(wire
@@
 			)
 		)
-		(pin "CS1" input
+		(pin "nCS1" input
 			(at 127 71.12 180)
 			(effects
@@
 			)
 		)
-		(pin "CS2" input
+		(pin "nCS2" input
 			(at 127 73.66 180)
 			(effects
@@
 			)
 		)
-		(pin "ADC1_CS" output
+		(pin "ADC1_nCS" output
 			(at 101.6 71.12 0)
 			(effects
@@
 			)
 		)
-		(pin "ADC2_CS" output
+		(pin "ADC2_nCS" output
 			(at 101.6 73.66 0)
 			(effects

Commit message: Final Updates:
- Mounting holes for an isolation shield
- 5V test-point to inject power
- Test signal input with resistor ladder
Parts:
- added H5, H6: MountingHole, MountingHole:MountingHole_3.5mm_Pad_Via, symbol Connectors:MountingHole
- renumbered H5 to H7, H6 to H8
Connections:
- net GND: now also H5.1, H6.1
Other:
- moved on the sheet: TP1, TP2, TP3
