File: KiCAD/Transmitter.kicad_sch (KiCad schematic)
At the start: 16 parts, among them U7 TPA6211A1DRBR

Commit message: Added title block and version text
Parts:
- renumbered C51 to C1, C52 to C2, C53 to C3, C54 to C4, C55 to C5, C56 to C6, C57 to C7, C58 to C8, R34 to R2, R35 to R3, R36 to R4, R37 to R5, TP8 to TP4, TP9 to TP5, U7 to U1
Other:
- company: (none) -> University of Cape Town
- title: (none) -> Transmitter
Changed lines of the file:
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@@
 	(generator_version "10.0")
 	(paper "A4")
+	(title_block
+		(title "Transmitter")
+		(date "2026-05-09")
+		(rev "v1.0")
+		(company "University of Cape Town")
+	)
 	(junction
 		(at 182.88 91.44)
@@
 		(dnp no)
 		(fields_autoplaced yes)
-		(property "Reference" "TP8"
+		(property "Reference" "TP4"
 			(at 170.18 48.7679 0)
 			(show_name no)
@@
 			(project "Sonar"
 				(path "/28f9d169-72cd-4bf2-894c-12741d733c98/d06a8764-b678-496b-8ef3-374055721279"
-					(reference "TP8")
+					(reference "TP4")
 					(unit 1)
 				)
@@
 		(in_pos_files yes)
 		(dnp no)
-		(property "Reference" "#PWR0112"
+		(property "Reference" "#PWR022"
 			(at 96.52 52.07 0)
 			(hide yes)
@@
 			(project "Sonar"
 				(path "/28f9d169-72cd-4bf2-894c-12741d733c98/d06a8764-b678-496b-8ef3-374055721279"
-					(reference "#PWR0112")
+					(reference "#PWR022")
 					(unit 1)
 				)
@@
 		(in_pos_files yes)
 		(dnp no)
-		(property "Reference" "#PWR0119"
+		(property "Reference" "#PWR029"
 			(at 124.46 133.35 0)
 			(hide yes)
@@
 			(project "Sonar"
 				(path "/28f9d169-72cd-4bf2-894c-12741d733c98/d06a8764-b678-496b-8ef3-374055721279"
-					(reference "#PWR0119")
+					(reference "#PWR029")
 					(unit 1)
 				)
@@
 		(dnp no)
 		(fields_autoplaced yes)
-		(property "Reference" "TP9"
+		(property "Reference" "TP5"
 			(at 170.18 64.0079 0)
 			(show_name no)
@@
 			(project "Sonar"
 				(path "/28f9d169-72cd-4bf2-894c-12741d733c98/d06a8764-b678-496b-8ef3-374055721279"
-					(reference "TP9")
+					(reference "TP5")
 					(unit 1)
 				)
@@
 		(dnp no)
 		(fields_autoplaced yes)
-		(property "Reference" "R36"
+		(property "Reference" "R4"
 			(at 88.9 85.09 90)
 			(show_name no)
@@
 			(project "Sonar"
 				(path "/28f9d169-72cd-4bf2-894c-12741d733c98/d06a8764-b678-496b-8ef3-374055721279"
-					(reference "R36")
+					(reference "R4")
 					(unit 1)
 				)
@@
 		(in_pos_files yes)
 		(dnp no)
-		(property "Reference" "U7"
+		(property "Reference" "U1"
 			(at 149.86 73.66 0)
 			(show_name no)
@@
 			(project "Sonar"
 				(path "/28f9d169-72cd-4bf2-894c-12741d733c98/d06a8764-b678-496b-8ef3-374055721279"
-					(reference "U7")
+					(reference "U1")
 					(unit 1)
 				)
@@
 		(dnp no)
 		(fields_autoplaced yes)
-		(property "Reference" "C54"
+		(property "Reference" "C4"
 			(at 104.14 72.39 90)
 			(show_name no)
@@
 			(project "Sonar"
 				(path "/28f9d169-72cd-4bf2-894c-12741d733c98/d06a8764-b678-496b-8ef3-374055721279"
-					(reference "C54")
+					(reference "C4")
 					(unit 1)
 				)
@@
 		(dnp no)
 		(fields_autoplaced yes)
-		(property "Reference" "C53"
+		(property "Reference" "C3"
 			(at 149.86 59.69 90)
 			(show_name no)
@@
 			(project "Sonar"
 				(path "/28f9d169-72cd-4bf2-894c-12741d733c98/d06a8764-b678-496b-8ef3-374055721279"
-					(reference "C53")
+					(reference "C3")
 					(unit 1)
 				)
@@
 		(dnp no)
 		(fields_autoplaced yes)
-		(property "Reference" "C57"
+		(property "Reference" "C7"
 			(at 180.34 114.2999 0)
 			(show_name no)
@@
 			(project "Sonar"
 				(path "/28f9d169-72cd-4bf2-894c-12741d733c98/d06a8764-b678-496b-8ef3-374055721279"
-					(reference "C57")
+					(reference "C7")
 					(unit 1)
 				)
@@
 		(dnp no)
 		(fields_autoplaced yes)
-		(property "Reference" "R34"
+		(property "Reference" "R2"
 			(at 88.9 72.39 90)
 			(show_name no)
@@
 			(project "Sonar"
 				(path "/28f9d169-72cd-4bf2-894c-12741d733c98/d06a8764-b678-496b-8ef3-374055721279"
-					(reference "R34")
+					(reference "R2")
 					(unit 1)
 				)
@@
 		(dnp no)
 		(fields_autoplaced yes)
-		(property "Reference" "C56"
+		(property "Reference" "C6"
 			(at 99.06 99.0599 0)
 			(show_name no)
@@
 			(project "Sonar"
 				(path "/28f9d169-72cd-4bf2-894c-12741d733c98/d06a8764-b678-496b-8ef3-374055721279"
-					(reference "C56")
+					(reference "C6")
 					(unit 1)
 				)
@@
 		(dnp no)
 		(fields_autoplaced yes)
-		(property "Reference" "C51"
+		(property "Reference" "C1"
 			(at 149.86 44.45 90)
 			(show_name no)
@@
 			(project "Sonar"
 				(path "/28f9d169-72cd-4bf2-894c-12741d733c98/d06a8764-b678-496b-8ef3-374055721279"
-					(reference "C51")
+					(reference "C1")
 					(unit 1)
 				)
@@
 		(in_pos_files yes)
 		(dnp no)
-		(property "Reference" "#PWR0116"
+		(property "Reference" "#PWR026"
 			(at 177.8 113.03 0)
 			(hide yes)
@@
 			(project "Sonar"
 				(path "/28f9d169-72cd-4bf2-894c-12741d733c98/d06a8764-b678-496b-8ef3-374055721279"
-					(reference "#PWR0116")
+					(reference "#PWR026")
 					(unit 1)
 				)
@@
 		(in_pos_files yes)
 		(dnp no)
-		(property "Reference" "#PWR0118"
+		(property "Reference" "#PWR028"
 			(at 177.8 130.81 0)
 			(hide yes)
@@
 			(project "Sonar"
 				(path "/28f9d169-72cd-4bf2-894c-12741d733c98/d06a8764-b678-496b-8ef3-374055721279"
-					(reference "#PWR0118")
+					(reference "#PWR028")
 					(unit 1)
 				)
@@
 		(in_pos_files yes)
 		(dnp no)
-		(property "Reference" "#PWR0115"
+		(property "Reference" "#PWR025"
 			(at 96.52 115.57 0)
 			(hide yes)
@@
 			(project "Sonar"
 				(path "/28f9d169-72cd-4bf2-894c-12741d733c98/d06a8764-b678-496b-8ef3-374055721279"
-					(reference "#PWR0115")
+					(reference "#PWR025")
 					(unit 1)
 				)
@@
 		(in_pos_files yes)
 		(dnp no)
-		(property "Reference" "#PWR0114"
+		(property "Reference" "#PWR024"
 			(at 74.93 81.28 0)
 			(hide yes)
@@
 			(project "Sonar"
 				(path "/28f9d169-72cd-4bf2-894c-12741d733c98/d06a8764-b678-496b-8ef3-374055721279"
-					(reference "#PWR0114")
+					(reference "#PWR024")
 					(unit 1)
 				)
@@
 		(dnp no)
 		(fields_autoplaced yes)
-		(property "Reference" "C55"
+		(property "Reference" "C5"
 			(at 104.14 85.09 90)
 			(show_name no)
@@
 			(project "Sonar"
 				(path "/28f9d169-72cd-4bf2-894c-12741d733c98/d06a8764-b678-496b-8ef3-374055721279"
-					(reference "C55")
+					(reference "C5")
 					(unit 1)
 				)
@@
 		(dnp no)
 		(fields_autoplaced yes)
-		(property "Reference" "#PWR0113"
+		(property "Reference" "#PWR023"
 			(at 166.37 78.74 0)
 			(hide yes)
@@
 			(project "Sonar"
 				(path "/28f9d169-72cd-4bf2-894c-12741d733c98/d06a8764-b678-496b-8ef3-374055721279"
-					(reference "#PWR0113")
+					(reference "#PWR023")
 					(unit 1)
 				)
@@
 		(dnp no)
 		(fields_autoplaced yes)
-		(property "Reference" "C58"
+		(property "Reference" "C8"
 			(at 127 116.8399 0)
 			(show_name no)
@@
 			(project "Sonar"
 				(path "/28f9d169-72cd-4bf2-894c-12741d733c98/d06a8764-b678-496b-8ef3-374055721279"
-					(reference "C58")
+					(reference "C8")
 					(unit 1)
 				)
@@
 		(dnp no)
 		(fields_autoplaced yes)
-		(property "Reference" "C52"
+		(property "Reference" "C2"
 			(at 99.06 63.4999 0)
 			(show_name no)
@@
 			(project "Sonar"
 				(path "/28f9d169-72cd-4bf2-894c-12741d733c98/d06a8764-b678-496b-8ef3-374055721279"
-					(reference "C52")
+					(reference "C2")
 					(unit 1)
 				)
@@
 		(dnp no)
 		(fields_autoplaced yes)
-		(property "Reference" "R35"
+		(property "Reference" "R3"
 			(at 116.84 72.39 90)
 			(show_name no)
@@
 			(project "Sonar"
 				(path "/28f9d169-72cd-4bf2-894c-12741d733c98/d06a8764-b678-496b-8ef3-374055721279"
-					(reference "R35")
+					(reference "R3")
 					(unit 1)
 				)
@@
 		(in_pos_files yes)
 		(dnp no)
-		(property "Reference" "#PWR0117"
+		(property "Reference" "#PWR027"
 			(at 170.18 130.81 0)
 			(hide yes)
@@
 			(project "Sonar"
 				(path "/28f9d169-72cd-4bf2-894c-12741d733c98/d06a8764-b678-496b-8ef3-374055721279"
-					(reference "#PWR0117")
+					(reference "#PWR027")
 					(unit 1)
 				)
@@
 		(dnp no)
 		(fields_autoplaced yes)
-		(property "Reference" "R37"
+		(property "Reference" "R5"
 			(at 116.84 85.09 90)
 			(show_name no)
@@
 			(project "Sonar"
 				(path "/28f9d169-72cd-4bf2-894c-12741d733c98/d06a8764-b678-496b-8ef3-374055721279"
-					(reference "R37")
+					(reference "R5")
 					(unit 1)
 				)

Commit message: Final Updates:
- Mounting holes for an isolation shield
- 5V test-point to inject power
- Test signal input with resistor ladder
Parts:
- renumbered TP4 to TP5, TP5 to TP6
Changed lines of the file:
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@@
 		(dnp no)
 		(fields_autoplaced yes)
-		(property "Reference" "TP4"
+		(property "Reference" "TP5"
 			(at 170.18 48.7679 0)
 			(show_name no)
@@
 			(project "Sonar"
 				(path "/28f9d169-72cd-4bf2-894c-12741d733c98/d06a8764-b678-496b-8ef3-374055721279"
-					(reference "TP4")
+					(reference "TP5")
 					(unit 1)
 				)
@@
 		(in_pos_files yes)
 		(dnp no)
-		(property "Reference" "#PWR022"
+		(property "Reference" "#PWR024"
 			(at 96.52 52.07 0)
 			(hide yes)
@@
 			(project "Sonar"
 				(path "/28f9d169-72cd-4bf2-894c-12741d733c98/d06a8764-b678-496b-8ef3-374055721279"
-					(reference "#PWR022")
+					(reference "#PWR024")
 					(unit 1)
 				)
@@
 		(in_pos_files yes)
 		(dnp no)
-		(property "Reference" "#PWR029"
+		(property "Reference" "#PWR031"
 			(at 124.46 133.35 0)
 			(hide yes)
@@
 			(project "Sonar"
 				(path "/28f9d169-72cd-4bf2-894c-12741d733c98/d06a8764-b678-496b-8ef3-374055721279"
-					(reference "#PWR029")
+					(reference "#PWR031")
 					(unit 1)
 				)
@@
 		(dnp no)
 		(fields_autoplaced yes)
-		(property "Reference" "TP5"
+		(property "Reference" "TP6"
 			(at 170.18 64.0079 0)
 			(show_name no)
@@
 			(project "Sonar"
 				(path "/28f9d169-72cd-4bf2-894c-12741d733c98/d06a8764-b678-496b-8ef3-374055721279"
-					(reference "TP5")
+					(reference "TP6")
 					(unit 1)
 				)
@@
 		(in_pos_files yes)
 		(dnp no)
-		(property "Reference" "#PWR026"
+		(property "Reference" "#PWR028"
 			(at 177.8 113.03 0)
 			(hide yes)
@@
 			(project "Sonar"
 				(path "/28f9d169-72cd-4bf2-894c-12741d733c98/d06a8764-b678-496b-8ef3-374055721279"
-					(reference "#PWR026")
+					(reference "#PWR028")
 					(unit 1)
 				)
@@
 		(in_pos_files yes)
 		(dnp no)
-		(property "Reference" "#PWR028"
+		(property "Reference" "#PWR030"
 			(at 177.8 130.81 0)
 			(hide yes)
@@
 			(project "Sonar"
 				(path "/28f9d169-72cd-4bf2-894c-12741d733c98/d06a8764-b678-496b-8ef3-374055721279"
-					(reference "#PWR028")
+					(reference "#PWR030")
 					(unit 1)
 				)
@@
 		(in_pos_files yes)
 		(dnp no)
-		(property "Reference" "#PWR025"
+		(property "Reference" "#PWR027"
 			(at 96.52 115.57 0)
 			(hide yes)
@@
 			(project "Sonar"
 				(path "/28f9d169-72cd-4bf2-894c-12741d733c98/d06a8764-b678-496b-8ef3-374055721279"
-					(reference "#PWR025")
+					(reference "#PWR027")
 					(unit 1)
 				)
@@
 		(in_pos_files yes)
 		(dnp no)
-		(property "Reference" "#PWR024"
+		(property "Reference" "#PWR026"
 			(at 74.93 81.28 0)
 			(hide yes)
@@
 			(project "Sonar"
 				(path "/28f9d169-72cd-4bf2-894c-12741d733c98/d06a8764-b678-496b-8ef3-374055721279"
-					(reference "#PWR024")
+					(reference "#PWR026")
 					(unit 1)
 				)
@@
 		(dnp no)
 		(fields_autoplaced yes)
-		(property "Reference" "#PWR023"
+		(property "Reference" "#PWR025"
 			(at 166.37 78.74 0)
 			(hide yes)
@@
 			(project "Sonar"
 				(path "/28f9d169-72cd-4bf2-894c-12741d733c98/d06a8764-b678-496b-8ef3-374055721279"
-					(reference "#PWR023")
+					(reference "#PWR025")
 					(unit 1)
 				)
@@
 		(in_pos_files yes)
 		(dnp no)
-		(property "Reference" "#PWR027"
+		(property "Reference" "#PWR029"
 			(at 170.18 130.81 0)
 			(hide yes)
@@
 			(project "Sonar"
 				(path "/28f9d169-72cd-4bf2-894c-12741d733c98/d06a8764-b678-496b-8ef3-374055721279"
-					(reference "#PWR027")
+					(reference "#PWR029")
 					(unit 1)
 				)
