File: KiCAD/Transmitter.kicad_sch (KiCad schematic)
At the start: 16 parts, among them U1 TPA6211A1DRBR

Commit message: Updated speaker and microphone library path to "Transducers"
Parts:
- LS1: symbol Audio:AS03208MS-3-R -> Transducers:AS03208MS-3-R
Changed lines of the file:
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@@
 	)
 	(symbol
-		(lib_id "Audio:AS03208MS-3-R")
+		(lib_id "Transducers:AS03208MS-3-R")
 		(at 187.96 88.9 0)
 		(unit 1)

Commit message: Changed 100pF and 100nF to AVX parts, and gave TPA6211 a pin-1 dot
Parts:
- C1, C3: MPN GCG1885G1H101JA01D -> KGM15AR71H101K; Manufacturer Murata -> KYOCERA AVX; SPN 81-GCG1885G1H101JA1D -> 581-KGM15AR71H101KT
Changed lines of the file:
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@@
 			)
 		)
-		(property "Manufacturer" "Murata"
+		(property "Manufacturer" "KYOCERA AVX"
 			(at 144.78 55.88 0)
 			(hide yes)
@@
 			)
 		)
-		(property "MPN" "GCG1885G1H101JA01D"
+		(property "MPN" "KGM15AR71H101K"
 			(at 147.32 55.88 0)
 			(hide yes)
@@
 			)
 		)
-		(property "SPN" "81-GCG1885G1H101JA1D"
+		(property "SPN" "581-KGM15AR71H101KT"
 			(at 152.4 55.88 0)
 			(hide yes)
@@
 			)
 		)
-		(property "Manufacturer" "Murata"
+		(property "Manufacturer" "KYOCERA AVX"
 			(at 144.78 40.64 0)
 			(hide yes)
@@
 			)
 		)
-		(property "MPN" "GCG1885G1H101JA01D"
+		(property "MPN" "KGM15AR71H101K"
 			(at 147.32 40.64 0)
 			(hide yes)
@@
 			)
 		)
-		(property "SPN" "81-GCG1885G1H101JA1D"
+		(property "SPN" "581-KGM15AR71H101KT"
 			(at 152.4 40.64 0)
 			(hide yes)
