File: KiCAD/MicArray.kicad_sch (KiCad schematic)
At the start: 64 parts, among them SW1 CrossBar, SW10 CrossBar, SW11 CrossBar, SW12 CrossBar, SW13 CrossBar, SW14 CrossBar, SW15 CrossBar, SW16 CrossBar, SW17 CrossBar, SW18 CrossBar, SW19 CrossBar, SW2 CrossBar, SW20 CrossBar, SW21 CrossBar, SW22 CrossBar, SW23 CrossBar, SW24 CrossBar, SW25 CrossBar, SW26 CrossBar, SW27 CrossBar, SW28 CrossBar, SW29 CrossBar, SW3 CrossBar, SW30 CrossBar, SW31 CrossBar, SW32 CrossBar, SW33 CrossBar, SW34 CrossBar, SW35 CrossBar, SW36 CrossBar, SW37 CrossBar, SW38 CrossBar, SW39 CrossBar, SW4 CrossBar, SW40 CrossBar, SW41 CrossBar, SW42 CrossBar, SW43 CrossBar, SW44 CrossBar, SW45 CrossBar, SW46 CrossBar, SW47 CrossBar, SW48 CrossBar, SW49 CrossBar, SW5 CrossBar, SW50 CrossBar, SW51 CrossBar, SW52 CrossBar, SW53 CrossBar, SW54 CrossBar, SW55 CrossBar, SW56 CrossBar, SW57 CrossBar, SW58 CrossBar, SW59 CrossBar, SW6 CrossBar, SW60 CrossBar, SW61 CrossBar, SW62 CrossBar, SW63 CrossBar, SW64 CrossBar, SW7 CrossBar, SW8 CrossBar, SW9 CrossBar

Commit message: Finished routing
Parts:
- SW1, SW10, SW11, SW12, SW13, SW14, SW15, SW16, SW17, SW18, SW19, SW2, SW20, SW21, SW22, SW23, SW24, SW25, SW26, SW27, SW28, SW29, SW3, SW30, SW31, SW32, SW33, SW34, SW35, SW36, SW37, SW38, SW39, SW4, SW40, SW41, SW42, SW43, SW44, SW45, SW46, SW47, SW48, SW49, SW5, SW50, SW51, SW52, SW53, SW54, SW55, SW56, SW57, SW58, SW59, SW6, SW60, SW61, SW62, SW63, SW64, SW7, SW8, SW9: footprint (none) -> Sonar:CrossBar_2x2
Connections:
- net Mic10/OUT: now also SW11.8 (OUTPUT_(+)), SW3.3 (OUTPUT_(+)); no longer SW11.3 (OUTPUT_(+)), SW19.8 (OUTPUT_(+))
- net Mic11/OUT: now also SW12.8 (OUTPUT_(+)), SW4.3 (OUTPUT_(+)); no longer SW12.3 (OUTPUT_(+)), SW20.8 (OUTPUT_(+))
- net Mic12/OUT: now also SW13.8 (OUTPUT_(+)), SW5.3 (OUTPUT_(+)); no longer SW13.3 (OUTPUT_(+)), SW21.8 (OUTPUT_(+))
- net Mic13/OUT: now also SW14.8 (OUTPUT_(+)), SW6.3 (OUTPUT_(+)); no longer SW14.3 (OUTPUT_(+)), SW22.8 (OUTPUT_(+))
- net Mic14/OUT: now also SW15.8 (OUTPUT_(+)), SW7.3 (OUTPUT_(+)); no longer SW15.3 (OUTPUT_(+)), SW23.8 (OUTPUT_(+))
- net Mic15/OUT: now also SW16.8 (OUTPUT_(+)), SW8.3 (OUTPUT_(+)); no longer SW16.3 (OUTPUT_(+)), SW24.8 (OUTPUT_(+))
- net Mic16/OUT: now also SW17.8 (OUTPUT_(+)), SW9.3 (OUTPUT_(+)); no longer SW25.3 (OUTPUT_(+)), SW33.8 (OUTPUT_(+))
- net Mic17/OUT: now also SW10.3 (OUTPUT_(+)), SW18.8 (OUTPUT_(+)); no longer SW26.3 (OUTPUT_(+)), SW34.8 (OUTPUT_(+))
- net Mic18/OUT: now also SW11.3 (OUTPUT_(+)), SW19.8 (OUTPUT_(+)); no longer SW27.3 (OUTPUT_(+)), SW35.8 (OUTPUT_(+))
- net Mic19/OUT: now also SW12.3 (OUTPUT_(+)), SW20.8 (OUTPUT_(+)); no longer SW28.3 (OUTPUT_(+)), SW36.8 (OUTPUT_(+))
- net Mic20/OUT: now also SW13.3 (OUTPUT_(+)), SW21.8 (OUTPUT_(+)); no longer SW29.3 (OUTPUT_(+)), SW37.8 (OUTPUT_(+))
- net Mic21/OUT: now also SW14.3 (OUTPUT_(+)), SW22.8 (OUTPUT_(+)); no longer SW30.3 (OUTPUT_(+)), SW38.8 (OUTPUT_(+))
- net Mic22/OUT: now also SW15.3 (OUTPUT_(+)), SW23.8 (OUTPUT_(+)); no longer SW31.3 (OUTPUT_(+)), SW39.8 (OUTPUT_(+))
- net Mic23/OUT: now also SW16.3 (OUTPUT_(+)), SW24.8 (OUTPUT_(+)); no longer SW32.3 (OUTPUT_(+)), SW40.8 (OUTPUT_(+))
- net Mic24/OUT: now also SW17.3 (OUTPUT_(+)), SW25.8 (OUTPUT_(+)); no longer SW41.3 (OUTPUT_(+)), SW49.8 (OUTPUT_(+))
- net Mic25/OUT: now also SW18.3 (OUTPUT_(+)), SW26.8 (OUTPUT_(+)); no longer SW42.3 (OUTPUT_(+)), SW50.8 (OUTPUT_(+))
- net Mic26/OUT: now also SW19.3 (OUTPUT_(+)), SW27.8 (OUTPUT_(+)); no longer SW43.3 (OUTPUT_(+)), SW51.8 (OUTPUT_(+))
- net Mic27/OUT: now also SW20.3 (OUTPUT_(+)), SW28.8 (OUTPUT_(+)); no longer SW44.3 (OUTPUT_(+)), SW52.8 (OUTPUT_(+))
- net Mic28/OUT: now also SW21.3 (OUTPUT_(+)), SW29.8 (OUTPUT_(+)); no longer SW45.3 (OUTPUT_(+)), SW53.8 (OUTPUT_(+))
- net Mic29/OUT: now also SW22.3 (OUTPUT_(+)), SW30.8 (OUTPUT_(+)); no longer SW46.3 (OUTPUT_(+)), SW54.8 (OUTPUT_(+))
- net Mic30/OUT: now also SW23.3 (OUTPUT_(+)), SW31.8 (OUTPUT_(+)); no longer SW47.3 (OUTPUT_(+)), SW55.8 (OUTPUT_(+))
- net Mic31/OUT: now also SW24.3 (OUTPUT_(+)), SW32.8 (OUTPUT_(+)); no longer SW48.3 (OUTPUT_(+)), SW56.8 (OUTPUT_(+))
- net Mic32/OUT: now also SW25.3 (OUTPUT_(+)), SW33.8 (OUTPUT_(+)); no longer SW1.3 (OUTPUT_(+)), SW9.8 (OUTPUT_(+))
- net Mic33/OUT: now also SW26.3 (OUTPUT_(+)), SW34.8 (OUTPUT_(+)); no longer SW10.8 (OUTPUT_(+)), SW2.3 (OUTPUT_(+))
- net Mic34/OUT: now also SW27.3 (OUTPUT_(+)), SW35.8 (OUTPUT_(+)); no longer SW11.8 (OUTPUT_(+)), SW3.3 (OUTPUT_(+))
- net Mic35/OUT: now also SW28.3 (OUTPUT_(+)), SW36.8 (OUTPUT_(+)); no longer SW12.8 (OUTPUT_(+)), SW4.3 (OUTPUT_(+))
- net Mic36/OUT: now also SW29.3 (OUTPUT_(+)), SW37.8 (OUTPUT_(+)); no longer SW13.8 (OUTPUT_(+)), SW5.3 (OUTPUT_(+))
- net Mic37/OUT: now also SW30.3 (OUTPUT_(+)), SW38.8 (OUTPUT_(+)); no longer SW14.8 (OUTPUT_(+)), SW6.3 (OUTPUT_(+))
- net Mic38/OUT: now also SW31.3 (OUTPUT_(+)), SW39.8 (OUTPUT_(+)); no longer SW15.8 (OUTPUT_(+)), SW7.3 (OUTPUT_(+))
- net Mic39/OUT: now also SW32.3 (OUTPUT_(+)), SW40.8 (OUTPUT_(+)); no longer SW16.8 (OUTPUT_(+)), SW8.3 (OUTPUT_(+))
- net Mic40/OUT: now also SW33.3 (OUTPUT_(+)), SW41.8 (OUTPUT_(+)); no longer SW17.3 (OUTPUT_(+)), SW25.8 (OUTPUT_(+))
- net Mic41/OUT: now also SW34.3 (OUTPUT_(+)), SW42.8 (OUTPUT_(+)); no longer SW18.3 (OUTPUT_(+)), SW26.8 (OUTPUT_(+))
- net Mic42/OUT: now also SW35.3 (OUTPUT_(+)), SW43.8 (OUTPUT_(+)); no longer SW19.3 (OUTPUT_(+)), SW27.8 (OUTPUT_(+))
- net Mic43/OUT: now also SW36.3 (OUTPUT_(+)), SW44.8 (OUTPUT_(+)); no longer SW20.3 (OUTPUT_(+)), SW28.8 (OUTPUT_(+))
- net Mic44/OUT: now also SW37.3 (OUTPUT_(+)), SW45.8 (OUTPUT_(+)); no longer SW21.3 (OUTPUT_(+)), SW29.8 (OUTPUT_(+))
- net Mic45/OUT: now also SW38.3 (OUTPUT_(+)), SW46.8 (OUTPUT_(+)); no longer SW22.3 (OUTPUT_(+)), SW30.8 (OUTPUT_(+))
- net Mic46/OUT: now also SW39.3 (OUTPUT_(+)), SW47.8 (OUTPUT_(+)); no longer SW23.3 (OUTPUT_(+)), SW31.8 (OUTPUT_(+))
- net Mic47/OUT: now also SW40.3 (OUTPUT_(+)), SW48.8 (OUTPUT_(+)); no longer SW24.3 (OUTPUT_(+)), SW32.8 (OUTPUT_(+))
- net Mic48/OUT: now also SW41.3 (OUTPUT_(+)), SW49.8 (OUTPUT_(+)); no longer SW33.3 (OUTPUT_(+)), SW41.8 (OUTPUT_(+))
- net Mic49/OUT: now also SW42.3 (OUTPUT_(+)), SW50.8 (OUTPUT_(+)); no longer SW34.3 (OUTPUT_(+)), SW42.8 (OUTPUT_(+))
- net Mic50/OUT: now also SW43.3 (OUTPUT_(+)), SW51.8 (OUTPUT_(+)); no longer SW35.3 (OUTPUT_(+)), SW43.8 (OUTPUT_(+))
- net Mic51/OUT: now also SW44.3 (OUTPUT_(+)), SW52.8 (OUTPUT_(+)); no longer SW36.3 (OUTPUT_(+)), SW44.8 (OUTPUT_(+))
- net Mic52/OUT: now also SW45.3 (OUTPUT_(+)), SW53.8 (OUTPUT_(+)); no longer SW37.3 (OUTPUT_(+)), SW45.8 (OUTPUT_(+))
- net Mic53/OUT: now also SW46.3 (OUTPUT_(+)), SW54.8 (OUTPUT_(+)); no longer SW38.3 (OUTPUT_(+)), SW46.8 (OUTPUT_(+))
- net Mic54/OUT: now also SW47.3 (OUTPUT_(+)), SW55.8 (OUTPUT_(+)); no longer SW39.3 (OUTPUT_(+)), SW47.8 (OUTPUT_(+))
- net Mic55/OUT: now also SW48.3 (OUTPUT_(+)), SW56.8 (OUTPUT_(+)); no longer SW40.3 (OUTPUT_(+)), SW48.8 (OUTPUT_(+))
- net Mic8/OUT: now also SW1.3 (OUTPUT_(+)), SW9.8 (OUTPUT_(+)); no longer SW17.8 (OUTPUT_(+)), SW9.3 (OUTPUT_(+))
- net Mic9/OUT: now also SW10.8 (OUTPUT_(+)), SW2.3 (OUTPUT_(+)); no longer SW10.3 (OUTPUT_(+)), SW18.8 (OUTPUT_(+))

Commit message: Added a debug header
Connections:
- net CH1: now also SW60.3 (OUTPUT_(+)); no longer SW57.3 (OUTPUT_(+))
- net CH10: now also SW64.4 (GND_(-)); no longer SW61.4 (GND_(-))
- net CH11: now also SW63.3 (OUTPUT_(+)); no longer SW62.3 (OUTPUT_(+))
- net CH12: now also SW63.4 (GND_(-)); no longer SW62.4 (GND_(-))
- net CH13: now also SW62.3 (OUTPUT_(+)); no longer SW63.3 (OUTPUT_(+))
- net CH14: now also SW62.4 (GND_(-)); no longer SW63.4 (GND_(-))
- net CH15: now also SW61.3 (OUTPUT_(+)); no longer SW64.3 (OUTPUT_(+))
- net CH16: now also SW61.4 (GND_(-)); no longer SW64.4 (GND_(-))
- net CH2: now also SW60.4 (GND_(-)); no longer SW57.4 (GND_(-))
- net CH3: now also SW59.3 (OUTPUT_(+)); no longer SW58.3 (OUTPUT_(+))
- net CH4: now also SW59.4 (GND_(-)); no longer SW58.4 (GND_(-))
- net CH5: now also SW58.3 (OUTPUT_(+)); no longer SW59.3 (OUTPUT_(+))
- net CH6: now also SW58.4 (GND_(-)); no longer SW59.4 (GND_(-))
- net CH7: now also SW57.3 (OUTPUT_(+)); no longer SW60.3 (OUTPUT_(+))
- net CH8: now also SW57.4 (GND_(-)); no longer SW60.4 (GND_(-))
- net CH9: now also SW64.3 (OUTPUT_(+)); no longer SW61.3 (OUTPUT_(+))
Changed lines of the file:
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@@
 	(hierarchical_label "CH8"
+		(shape output)
+		(at 48.26 233.68 270)
+		(effects
+			(font
+				(size 1.27 1.27)
+			)
+			(justify right)
+		)
+	)
+	(hierarchical_label "CH5"
+		(shape output)
+		(at 91.44 233.68 270)
+		(effects
+			(font
+				(size 1.27 1.27)
+			)
+			(justify right)
+		)
+	)
+	(hierarchical_label "CH2"
 		(shape output)
 		(at 193.04 233.68 270)
@@
 		)
 	)
-	(hierarchical_label "CH5"
+	(hierarchical_label "CH6"
+		(shape output)
+		(at 96.52 233.68 270)
+		(effects
+			(font
+				(size 1.27 1.27)
+			)
+			(justify right)
+		)
+	)
+	(hierarchical_label "CH4"
+		(shape output)
+		(at 144.78 233.68 270)
+		(effects
+			(font
+				(size 1.27 1.27)
+			)
+			(justify right)
+		)
+	)
+	(hierarchical_label "CH1"
+		(shape output)
+		(at 187.96 233.68 270)
+		(effects
+			(font
+				(size 1.27 1.27)
+			)
+			(justify right)
+		)
+	)
+	(hierarchical_label "CH14"
+		(shape output)
+		(at 289.56 233.68 270)
+		(effects
+			(font
+				(size 1.27 1.27)
+			)
+			(justify right)
+		)
+	)
+	(hierarchical_label "CH16"
+		(shape output)
+		(at 241.3 233.68 270)
+		(effects
+			(font
+				(size 1.27 1.27)
+			)
+			(justify right)
+		)
+	)
+	(hierarchical_label "CH13"
+		(shape output)
+		(at 284.48 233.68 270)
+		(effects
+			(font
+				(size 1.27 1.27)
+			)
+			(justify right)
+		)
+	)
+	(hierarchical_label "CH12"
+		(shape output)
+		(at 337.82 233.68 270)
+		(effects
+			(font
+				(size 1.27 1.27)
+			)
+			(justify right)
+		)
+	)
+	(hierarchical_label "CH3"
 		(shape output)
 		(at 139.7 233.68 270)
@@
 		)
 	)
-	(hierarchical_label "CH2"
+	(hierarchical_label "CH15"
 		(shape output)
-		(at 48.26 233.68 270)
+		(at 236.22 233.68 270)
 		(effects
 			(font
@@
 		)
 	)
-	(hierarchical_label "CH6"
-		(shape output)
-		(at 144.78 233.68 270)
-		(effects
-			(font
-				(size 1.27 1.27)
-			)
-			(justify right)
-		)
-	)
-	(hierarchical_label "CH4"
-		(shape output)
-		(at 96.52 233.68 270)
-		(effects
-			(font
-				(size 1.27 1.27)
-			)
-			(justify right)
-		)
-	)
-	(hierarchical_label "CH1"
+	(hierarchical_label "CH7"
 		(shape output)
 		(at 43.18 233.68 270)
@@
 		)
 	)
-	(hierarchical_label "CH14"
+	(hierarchical_label "CH9"
 		(shape output)
-		(at 337.82 233.68 270)
+		(at 381 233.68 270)
 		(effects
 			(font
@@
 		)
 	)
-	(hierarchical_label "CH16"
+	(hierarchical_label "CH10"
 		(shape output)
 		(at 386.08 233.68 270)
@@
 		)
 	)
-	(hierarchical_label "CH13"
+	(hierarchical_label "CH11"
 		(shape output)
 		(at 332.74 233.68 270)
 		(effects
 			(font
-				(size 1.27 1.27)
-			)
-			(justify right)
-		)
-	)
-	(hierarchical_label "CH12"
-		(shape output)
-		(at 289.56 233.68 270)
-		(effects
-			(font
-				(size 1.27 1.27)
-			)
-			(justify right)
-		)
-	)
-	(hierarchical_label "CH3"
-		(shape output)
-		(at 91.44 233.68 270)
-		(effects
-			(font
-				(size 1.27 1.27)
-			)
-			(justify right)
-		)
-	)
-	(hierarchical_label "CH15"
-		(shape output)
-		(at 381 233.68 270)
-		(effects
-			(font
-				(size 1.27 1.27)
-			)
-			(justify right)
-		)
-	)
-	(hierarchical_label "CH7"
-		(shape output)
-		(at 187.96 233.68 270)
-		(effects
-			(font
-				(size 1.27 1.27)
-			)
-			(justify right)
-		)
-	)
-	(hierarchical_label "CH9"
-		(shape output)
-		(at 236.22 233.68 270)
-		(effects
-			(font
-				(size 1.27 1.27)
-			)
-			(justify right)
-		)
-	)
-	(hierarchical_label "CH10"
-		(shape output)
-		(at 241.3 233.68 270)
-		(effects
-			(font
-				(size 1.27 1.27)
-			)
-			(justify right)
-		)
-	)
-	(hierarchical_label "CH11"
-		(shape output)
-		(at 284.48 233.68 270)
-		(effects
-			(font

Commit message: Moved the microphone RL to per-channel instead of per-mic
Parts:
- added MK1, MK10, MK11, MK12, MK13, MK14, MK15, MK16, MK17, MK18, MK19, MK2, MK20, MK21, MK22, MK23, MK24, MK25, MK26, MK27, MK28, MK29, MK3, MK30, MK31, MK32, MK33, MK34, MK35, MK36, MK37, MK38, MK39, MK4, MK40, MK41, MK42, MK43, MK44, MK45, MK46, MK47, MK48, MK49, MK5, MK50, MK51, MK52, MK53, MK54, MK55, MK56, MK57, MK58, MK59, MK6, MK60, MK61, MK62, MK63, MK64, MK7, MK8, MK9: CMEJ-0415-42-P, SamacSys_Parts:CMEJ041542P, symbol Sensors:CMEJ-0415-42-P
Connections:
- net Mic0/OUT: no longer names the net of SW1.8 (OUTPUT_(+))
- net Mic0/OUT: now also MK1.1 (OUTPUT_(+))
- net Mic1/OUT: no longer names the net of SW2.8 (OUTPUT_(+))
- net Mic1/OUT: now also MK2.1 (OUTPUT_(+))
- net Mic10/OUT: no longer names the net of SW11.8 (OUTPUT_(+)), SW3.3 (OUTPUT_(+))
- net Mic10/OUT: now also MK11.1 (OUTPUT_(+))
- net Mic11/OUT: no longer names the net of SW12.8 (OUTPUT_(+)), SW4.3 (OUTPUT_(+))
- net Mic11/OUT: now also MK12.1 (OUTPUT_(+))
- net Mic12/OUT: no longer names the net of SW13.8 (OUTPUT_(+)), SW5.3 (OUTPUT_(+))
- net Mic12/OUT: now also MK13.1 (OUTPUT_(+))
- net Mic13/OUT: no longer names the net of SW14.8 (OUTPUT_(+)), SW6.3 (OUTPUT_(+))
- net Mic13/OUT: now also MK14.1 (OUTPUT_(+))
- net Mic14/OUT: no longer names the net of SW15.8 (OUTPUT_(+)), SW7.3 (OUTPUT_(+))
- net Mic14/OUT: now also MK15.1 (OUTPUT_(+))
- net Mic15/OUT: no longer names the net of SW16.8 (OUTPUT_(+)), SW8.3 (OUTPUT_(+))
- net Mic15/OUT: now also MK16.1 (OUTPUT_(+))
- net Mic16/OUT: no longer names the net of SW17.8 (OUTPUT_(+)), SW9.3 (OUTPUT_(+))
- net Mic16/OUT: now also MK17.1 (OUTPUT_(+))
- net Mic17/OUT: no longer names the net of SW10.3 (OUTPUT_(+)), SW18.8 (OUTPUT_(+))
- net Mic17/OUT: now also MK18.1 (OUTPUT_(+))
- net Mic18/OUT: no longer names the net of SW11.3 (OUTPUT_(+)), SW19.8 (OUTPUT_(+))
- net Mic18/OUT: now also MK19.1 (OUTPUT_(+))
- net Mic19/OUT: no longer names the net of SW12.3 (OUTPUT_(+)), SW20.8 (OUTPUT_(+))
- net Mic19/OUT: now also MK20.1 (OUTPUT_(+))
- net Mic2/OUT: no longer names the net of SW3.8 (OUTPUT_(+))
- net Mic2/OUT: now also MK3.1 (OUTPUT_(+))
- net Mic20/OUT: no longer names the net of SW13.3 (OUTPUT_(+)), SW21.8 (OUTPUT_(+))
- net Mic20/OUT: now also MK21.1 (OUTPUT_(+))
- net Mic21/OUT: no longer names the net of SW14.3 (OUTPUT_(+)), SW22.8 (OUTPUT_(+))
- net Mic21/OUT: now also MK22.1 (OUTPUT_(+))
- net Mic22/OUT: no longer names the net of SW15.3 (OUTPUT_(+)), SW23.8 (OUTPUT_(+))
- net Mic22/OUT: now also MK23.1 (OUTPUT_(+))
- net Mic23/OUT: no longer names the net of SW16.3 (OUTPUT_(+)), SW24.8 (OUTPUT_(+))
- net Mic23/OUT: now also MK24.1 (OUTPUT_(+))
- net Mic24/OUT: no longer names the net of SW17.3 (OUTPUT_(+)), SW25.8 (OUTPUT_(+))
- net Mic24/OUT: now also MK25.1 (OUTPUT_(+))
- net Mic25/OUT: no longer names the net of SW18.3 (OUTPUT_(+)), SW26.8 (OUTPUT_(+))
- net Mic25/OUT: now also MK26.1 (OUTPUT_(+))
- net Mic26/OUT: no longer names the net of SW19.3 (OUTPUT_(+)), SW27.8 (OUTPUT_(+))
- net Mic26/OUT: now also MK27.1 (OUTPUT_(+))
- net Mic27/OUT: no longer names the net of SW20.3 (OUTPUT_(+)), SW28.8 (OUTPUT_(+))
- net Mic27/OUT: now also MK28.1 (OUTPUT_(+))
- net Mic28/OUT: no longer names the net of SW21.3 (OUTPUT_(+)), SW29.8 (OUTPUT_(+))
- net Mic28/OUT: now also MK29.1 (OUTPUT_(+))
- net Mic29/OUT: no longer names the net of SW22.3 (OUTPUT_(+)), SW30.8 (OUTPUT_(+))
- net Mic29/OUT: now also MK30.1 (OUTPUT_(+))
- net Mic3/OUT: no longer names the net of SW4.8 (OUTPUT_(+))
- net Mic3/OUT: now also MK4.1 (OUTPUT_(+))
- net Mic30/OUT: no longer names the net of SW23.3 (OUTPUT_(+)), SW31.8 (OUTPUT_(+))
- net Mic30/OUT: now also MK31.1 (OUTPUT_(+))
- net Mic31/OUT: no longer names the net of SW24.3 (OUTPUT_(+)), SW32.8 (OUTPUT_(+))
- net Mic31/OUT: now also MK32.1 (OUTPUT_(+))
- net Mic32/OUT: no longer names the net of SW25.3 (OUTPUT_(+)), SW33.8 (OUTPUT_(+))
- net Mic32/OUT: now also MK33.1 (OUTPUT_(+))
- net Mic33/OUT: no longer names the net of SW26.3 (OUTPUT_(+)), SW34.8 (OUTPUT_(+))
- net Mic33/OUT: now also MK34.1 (OUTPUT_(+))
- net Mic34/OUT: no longer names the net of SW27.3 (OUTPUT_(+)), SW35.8 (OUTPUT_(+))
- net Mic34/OUT: now also MK35.1 (OUTPUT_(+))
- net Mic35/OUT: no longer names the net of SW28.3 (OUTPUT_(+)), SW36.8 (OUTPUT_(+))
- net Mic35/OUT: now also MK36.1 (OUTPUT_(+))
- net Mic36/OUT: no longer names the net of SW29.3 (OUTPUT_(+)), SW37.8 (OUTPUT_(+))
- net Mic36/OUT: now also MK37.1 (OUTPUT_(+))
- net Mic37/OUT: no longer names the net of SW30.3 (OUTPUT_(+)), SW38.8 (OUTPUT_(+))
- net Mic37/OUT: now also MK38.1 (OUTPUT_(+))
- net Mic38/OUT: no longer names the net of SW31.3 (OUTPUT_(+)), SW39.8 (OUTPUT_(+))
- net Mic38/OUT: now also MK39.1 (OUTPUT_(+))
- net Mic39/OUT: no longer names the net of SW32.3 (OUTPUT_(+)), SW40.8 (OUTPUT_(+))
- net Mic39/OUT: now also MK40.1 (OUTPUT_(+))
- net Mic4/OUT: no longer names the net of SW5.8 (OUTPUT_(+))
- net Mic4/OUT: now also MK5.1 (OUTPUT_(+))
- net Mic40/OUT: no longer names the net of SW33.3 (OUTPUT_(+)), SW41.8 (OUTPUT_(+))
- net Mic40/OUT: now also MK41.1 (OUTPUT_(+))
- net Mic41/OUT: no longer names the net of SW34.3 (OUTPUT_(+)), SW42.8 (OUTPUT_(+))
- net Mic41/OUT: now also MK42.1 (OUTPUT_(+))
- net Mic42/OUT: no longer names the net of SW35.3 (OUTPUT_(+)), SW43.8 (OUTPUT_(+))
- net Mic42/OUT: now also MK43.1 (OUTPUT_(+))
- net Mic43/OUT: no longer names the net of SW36.3 (OUTPUT_(+)), SW44.8 (OUTPUT_(+))
- net Mic43/OUT: now also MK44.1 (OUTPUT_(+))
- net Mic44/OUT: no longer names the net of SW37.3 (OUTPUT_(+)), SW45.8 (OUTPUT_(+))
- net Mic44/OUT: now also MK45.1 (OUTPUT_(+))
- net Mic45/OUT: no longer names the net of SW38.3 (OUTPUT_(+)), SW46.8 (OUTPUT_(+))
- net Mic45/OUT: now also MK46.1 (OUTPUT_(+))
- net Mic46/OUT: no longer names the net of SW39.3 (OUTPUT_(+)), SW47.8 (OUTPUT_(+))
- net Mic46/OUT: now also MK47.1 (OUTPUT_(+))
- net Mic47/OUT: no longer names the net of SW40.3 (OUTPUT_(+)), SW48.8 (OUTPUT_(+))
- net Mic47/OUT: now also MK48.1 (OUTPUT_(+))
- net Mic48/OUT: no longer names the net of SW41.3 (OUTPUT_(+)), SW49.8 (OUTPUT_(+))
- net Mic48/OUT: now also MK49.1 (OUTPUT_(+))
- net Mic49/OUT: no longer names the net of SW42.3 (OUTPUT_(+)), SW50.8 (OUTPUT_(+))
- net Mic49/OUT: now also MK50.1 (OUTPUT_(+))
- net Mic5/OUT: no longer names the net of SW6.8 (OUTPUT_(+))
- net Mic5/OUT: now also MK6.1 (OUTPUT_(+))
- net Mic50/OUT: no longer names the net of SW43.3 (OUTPUT_(+)), SW51.8 (OUTPUT_(+))
- net Mic50/OUT: now also MK51.1 (OUTPUT_(+))
- net Mic51/OUT: no longer names the net of SW44.3 (OUTPUT_(+)), SW52.8 (OUTPUT_(+))
- net Mic51/OUT: now also MK52.1 (OUTPUT_(+))
- net Mic52/OUT: no longer names the net of SW45.3 (OUTPUT_(+)), SW53.8 (OUTPUT_(+))
- net Mic52/OUT: now also MK53.1 (OUTPUT_(+))
- net Mic53/OUT: no longer names the net of SW46.3 (OUTPUT_(+)), SW54.8 (OUTPUT_(+))
- net Mic53/OUT: now also MK54.1 (OUTPUT_(+))
- net Mic54/OUT: no longer names the net of SW47.3 (OUTPUT_(+)), SW55.8 (OUTPUT_(+))
- net Mic54/OUT: now also MK55.1 (OUTPUT_(+))
- net Mic55/OUT: no longer names the net of SW48.3 (OUTPUT_(+)), SW56.8 (OUTPUT_(+))
- net Mic55/OUT: now also MK56.1 (OUTPUT_(+))
- net Mic56/OUT: no longer names the net of SW49.3 (OUTPUT_(+)), SW57.8 (OUTPUT_(+))
- net Mic56/OUT: now also MK57.1 (OUTPUT_(+))
- net Mic57/OUT: no longer names the net of SW50.3 (OUTPUT_(+)), SW58.8 (OUTPUT_(+))
- net Mic57/OUT: now also MK58.1 (OUTPUT_(+))
- net Mic58/OUT: no longer names the net of SW51.3 (OUTPUT_(+)), SW59.8 (OUTPUT_(+))
- net Mic58/OUT: now also MK59.1 (OUTPUT_(+))
- net Mic59/OUT: no longer names the net of SW52.3 (OUTPUT_(+)), SW60.8 (OUTPUT_(+))
- net Mic59/OUT: now also MK60.1 (OUTPUT_(+))
- net Mic6/OUT: no longer names the net of SW7.8 (OUTPUT_(+))
- net Mic6/OUT: now also MK7.1 (OUTPUT_(+))
- net Mic60/OUT: no longer names the net of SW53.3 (OUTPUT_(+)), SW61.8 (OUTPUT_(+))
- net Mic60/OUT: now also MK61.1 (OUTPUT_(+))
- net Mic61/OUT: no longer names the net of SW54.3 (OUTPUT_(+)), SW62.8 (OUTPUT_(+))
- net Mic61/OUT: now also MK62.1 (OUTPUT_(+))
- net Mic62/OUT: no longer names the net of SW55.3 (OUTPUT_(+)), SW63.8 (OUTPUT_(+))
- net Mic62/OUT: now also MK63.1 (OUTPUT_(+))
- net Mic63/OUT: no longer names the net of SW56.3 (OUTPUT_(+)), SW64.8 (OUTPUT_(+))
- net Mic63/OUT: now also MK64.1 (OUTPUT_(+))
- net Mic7/OUT: no longer names the net of SW8.8 (OUTPUT_(+))
- net Mic7/OUT: now also MK8.1 (OUTPUT_(+))
- net Mic8/OUT: no longer names the net of SW1.3 (OUTPUT_(+)), SW9.8 (OUTPUT_(+))
- net Mic8/OUT: now also MK9.1 (OUTPUT_(+))
- net Mic9/OUT: no longer names the net of SW10.8 (OUTPUT_(+)), SW2.3 (OUTPUT_(+))
- net Mic9/OUT: now also MK10.1 (OUTPUT_(+))
- new net GND: MK1.2 (GND_(-)), MK10.2 (GND_(-)), MK11.2 (GND_(-)), MK12.2 (GND_(-)), MK13.2 (GND_(-)), MK14.2 (GND_(-)), MK15.2 (GND_(-)), MK16.2 (GND_(-)), MK17.2 (GND_(-)), MK18.2 (GND_(-)), MK19.2 (GND_(-)), MK2.2 (GND_(-)), MK20.2 (GND_(-)), MK21.2 (GND_(-)), MK22.2 (GND_(-)), MK23.2 (GND_(-)), MK24.2 (GND_(-)), MK25.2 (GND_(-)), MK26.2 (GND_(-)), MK27.2 (GND_(-)), MK28.2 (GND_(-)), MK29.2 (GND_(-)), MK3.2 (GND_(-)), MK30.2 (GND_(-)), MK31.2 (GND_(-)), MK32.2 (GND_(-)), MK33.2 (GND_(-)), MK34.2 (GND_(-)), MK35.2 (GND_(-)), MK36.2 (GND_(-)), MK37.2 (GND_(-)), MK38.2 (GND_(-)), MK39.2 (GND_(-)), MK4.2 (GND_(-)), MK40.2 (GND_(-)), MK41.2 (GND_(-)), MK42.2 (GND_(-)), MK43.2 (GND_(-)), MK44.2 (GND_(-)), MK45.2 (GND_(-)), MK46.2 (GND_(-)), MK47.2 (GND_(-)), MK48.2 (GND_(-)), MK49.2 (GND_(-)), MK5.2 (GND_(-)), MK50.2 (GND_(-)), MK51.2 (GND_(-)), MK52.2 (GND_(-)), MK53.2 (GND_(-)), MK54.2 (GND_(-)), MK55.2 (GND_(-)), MK56.2 (GND_(-)), MK57.2 (GND_(-)), MK58.2 (GND_(-)), MK59.2 (GND_(-)), MK6.2 (GND_(-)), MK60.2 (GND_(-)), MK61.2 (GND_(-)), MK62.2 (GND_(-)), MK63.2 (GND_(-)), MK64.2 (GND_(-)), MK7.2 (GND_(-)), MK8.2 (GND_(-)), MK9.2 (GND_(-))
Other:
- removed sheet Mic0
- removed sheet Mic1
- removed sheet Mic10
- removed sheet Mic11
- removed sheet Mic12
- removed sheet Mic13
- removed sheet Mic14
- removed sheet Mic15
- removed sheet Mic16
- removed sheet Mic17
- removed sheet Mic18
- removed sheet Mic19
- removed sheet Mic2
- removed sheet Mic20
- removed sheet Mic21
- removed sheet Mic22
- removed sheet Mic23
- removed sheet Mic24
- removed sheet Mic25
- removed sheet Mic26
- removed sheet Mic27
- removed sheet Mic28
- removed sheet Mic29
- removed sheet Mic3
- removed sheet Mic30
- removed sheet Mic31
- removed sheet Mic32
- removed sheet Mic33
- removed sheet Mic34
- removed sheet Mic35
- removed sheet Mic36
- removed sheet Mic37
- removed sheet Mic38
- removed sheet Mic39
- removed sheet Mic4
- removed sheet Mic40
- removed sheet Mic41
- removed sheet Mic42
- removed sheet Mic43
- removed sheet Mic44
- removed sheet Mic45
- removed sheet Mic46
- removed sheet Mic47
- removed sheet Mic48
- removed sheet Mic49
- removed sheet Mic5
- removed sheet Mic50
- removed sheet Mic51
- removed sheet Mic52
- removed sheet Mic53
- removed sheet Mic54
- removed sheet Mic55
- removed sheet Mic56
- removed sheet Mic57
- removed sheet Mic58
- removed sheet Mic59
- removed sheet Mic6
- removed sheet Mic60
- removed sheet Mic61
- removed sheet Mic62
- removed sheet Mic63
- removed sheet Mic7
- removed sheet Mic8
- removed sheet Mic9
- moved on the sheet: SW1, SW10, SW11, SW12, SW13, SW14, SW15, SW16, SW17, SW18, SW19, SW2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

Commit message: Added title block and version text
Other:
- company: (none) -> University of Cape Town
- title: (none) -> Microphone Array

Commit message: Final Updates:
- Mounting holes for an isolation shield
- 5V test-point to inject power
- Test signal input with resistor ladder
Parts:
- added R10, R11, R12, R13, R14, R15, R16, R17, R18, R19, R20, R21, R6, R7, R8, R9: R0603_10R, Resistor_SMD:R_0603_1608Metric, symbol Resistors0603:R0603_10R
- added R22: R0603_3k6, Resistor_SMD:R_0603_1608Metric, symbol Resistors0603:R0603_3k6
- added TP7: Keystone_5014_Yellow, TestPoint:TestPoint_Keystone_5010-5014_Multipurpose, symbol Connectors:Keystone_5014_Yellow
Connections:
- net GND: now also R6.1
- net at SW24.5 (GND_(-)): now also R11.2, R12.1
- net at SW24.6 (OUTPUT_(+)): now also R10.2, R11.1
- net at SW32.5 (GND_(-)): now also R13.2, R14.1
- net at SW32.6 (OUTPUT_(+)): now also R12.2, R13.1
- net at SW8.5 (GND_(-)): now also R7.2, R8.1
- net at SW8.6 (OUTPUT_(+)): now also R6.2, R7.1
- net at SW56.5 (GND_(-)): now also R19.2, R20.1
- net at SW56.6 (OUTPUT_(+)): now also R18.2, R19.1
- net at SW16.5 (GND_(-)): now also R10.1, R9.2
- net at SW16.6 (OUTPUT_(+)): now also R8.2, R9.1
- net at SW64.5 (GND_(-)): now also R21.2, R22.1
- net at SW64.6 (OUTPUT_(+)): now also R20.2, R21.1
- net at SW40.5 (GND_(-)): now also R15.2, R16.1
- net at SW40.6 (OUTPUT_(+)): now also R14.2, R15.1
- net at SW48.5 (GND_(-)): now also R17.2, R18.1
- net at SW48.6 (OUTPUT_(+)): now also R16.2, R17.1
- new net: R22.2, TP7.1
Other:
- moved on the sheet: MK1, MK10, MK11, MK12, MK13, MK14, MK15, MK16, MK17, MK18, MK19, MK2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
