File: KiCAD/MicArray.kicad_sch (KiCad schematic)
At the start: 146 parts, among them SW1 CrossBar, SW10 CrossBar, SW11 CrossBar, SW12 CrossBar, SW13 CrossBar, SW14 CrossBar, SW15 CrossBar, SW16 CrossBar, SW17 CrossBar, SW18 CrossBar, SW19 CrossBar, SW2 CrossBar, SW20 CrossBar, SW21 CrossBar, SW22 CrossBar, SW23 CrossBar, SW24 CrossBar, SW25 CrossBar, SW26 CrossBar, SW27 CrossBar, SW28 CrossBar, SW29 CrossBar, SW3 CrossBar, SW30 CrossBar, SW31 CrossBar, SW32 CrossBar, SW33 CrossBar, SW34 CrossBar, SW35 CrossBar, SW36 CrossBar, SW37 CrossBar, SW38 CrossBar, SW39 CrossBar, SW4 CrossBar, SW40 CrossBar, SW41 CrossBar, SW42 CrossBar, SW43 CrossBar, SW44 CrossBar, SW45 CrossBar, SW46 CrossBar, SW47 CrossBar, SW48 CrossBar, SW49 CrossBar, SW5 CrossBar, SW50 CrossBar, SW51 CrossBar, SW52 CrossBar, SW53 CrossBar, SW54 CrossBar, SW55 CrossBar, SW56 CrossBar, SW57 CrossBar, SW58 CrossBar, SW59 CrossBar, SW6 CrossBar, SW60 CrossBar, SW61 CrossBar, SW62 CrossBar, SW63 CrossBar, SW64 CrossBar, SW7 CrossBar, SW8 CrossBar, SW9 CrossBar

Commit message: Updated speaker and microphone library path to "Transducers"
Parts:
- MK1, MK10, MK11, MK12, MK13, MK14, MK15, MK16, MK17, MK18, MK19, MK2, MK20, MK21, MK22, MK23, MK24, MK25, MK26, MK27, MK28, MK29, MK3, MK30, MK31, MK32, MK33, MK34, MK35, MK36, MK37, MK38, MK39, MK4, MK40, MK41, MK42, MK43, MK44, MK45, MK46, MK47, MK48, MK49, MK5, MK50, MK51, MK52, MK53, MK54, MK55, MK56, MK57, MK58, MK59, MK6, MK60, MK61, MK62, MK63, MK64, MK7, MK8, MK9: symbol Sensors:CMEJ-0415-42-P -> Transducers:CMEJ-0415-42-P
Changed lines of the file:
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@@
 	)
 	(symbol
-		(lib_id "Sensors:CMEJ-0415-42-P")
+		(lib_id "Transducers:CMEJ-0415-42-P")
 		(at 99.06 180.34 0)
 		(mirror y)
@@
 	)
 	(symbol
-		(lib_id "Sensors:CMEJ-0415-42-P")
+		(lib_id "Transducers:CMEJ-0415-42-P")
 		(at 388.62 256.54 0)
 		(mirror y)
@@
 	)
 	(symbol
-		(lib_id "Sensors:CMEJ-0415-42-P")
+		(lib_id "Transducers:CMEJ-0415-42-P")
 		(at 99.06 256.54 0)
 		(mirror y)
@@
 	)
 	(symbol
-		(lib_id "Sensors:CMEJ-0415-42-P")
+		(lib_id "Transducers:CMEJ-0415-42-P")
 		(at 388.62 154.94 0)
 		(mirror y)
@@
 	)
 	(symbol
-		(lib_id "Sensors:CMEJ-0415-42-P")
+		(lib_id "Transducers:CMEJ-0415-42-P")
 		(at 388.62 231.14 0)
 		(mirror y)
@@
 	)
 	(symbol
-		(lib_id "Sensors:CMEJ-0415-42-P")
+		(lib_id "Transducers:CMEJ-0415-42-P")
 		(at 436.88 129.54 0)
 		(mirror y)
@@
 	)
 	(symbol
-		(lib_id "Sensors:CMEJ-0415-42-P")
+		(lib_id "Transducers:CMEJ-0415-42-P")
 		(at 99.06 129.54 0)
 		(mirror y)
@@
 	)
 	(symbol
-		(lib_id "Sensors:CMEJ-0415-42-P")
+		(lib_id "Transducers:CMEJ-0415-42-P")
 		(at 147.32 205.74 0)
 		(mirror y)
@@
 	)
 	(symbol
-		(lib_id "Sensors:CMEJ-0415-42-P")
+		(lib_id "Transducers:CMEJ-0415-42-P")
 		(at 436.88 104.14 0)
 		(mirror y)
@@
 	)
 	(symbol
-		(lib_id "Sensors:CMEJ-0415-42-P")
+		(lib_id "Transducers:CMEJ-0415-42-P")
 		(at 243.84 256.54 0)
 		(mirror y)
@@
 	)
 	(symbol
-		(lib_id "Sensors:CMEJ-0415-42-P")
+		(lib_id "Transducers:CMEJ-0415-42-P")
 		(at 436.88 256.54 0)
 		(mirror y)
@@
 	)
 	(symbol
-		(lib_id "Sensors:CMEJ-0415-42-P")
+		(lib_id "Transducers:CMEJ-0415-42-P")
 		(at 195.58 256.54 0)
 		(mirror y)
@@
 	)
 	(symbol
-		(lib_id "Sensors:CMEJ-0415-42-P")
+		(lib_id "Transducers:CMEJ-0415-42-P")
 		(at 340.36 180.34 0)
 		(mirror y)
@@
 	)
 	(symbol
-		(lib_id "Sensors:CMEJ-0415-42-P")
+		(lib_id "Transducers:CMEJ-0415-42-P")
 		(at 436.88 78.74 0)
 		(mirror y)
@@
 	)
 	(symbol
-		(lib_id "Sensors:CMEJ-0415-42-P")
+		(lib_id "Transducers:CMEJ-0415-42-P")
 		(at 147.32 78.74 0)
 		(mirror y)
@@
 	)
 	(symbol
-		(lib_id "Sensors:CMEJ-0415-42-P")
+		(lib_id "Transducers:CMEJ-0415-42-P")
 		(at 99.06 154.94 0)
 		(mirror y)
@@
 	)
 	(symbol
-		(lib_id "Sensors:CMEJ-0415-42-P")
+		(lib_id "Transducers:CMEJ-0415-42-P")
 		(at 195.58 129.54 0)
 		(mirror y)
@@
 	)
 	(symbol
-		(lib_id "Sensors:CMEJ-0415-42-P")
+		(lib_id "Transducers:CMEJ-0415-42-P")
 		(at 147.32 129.54 0)
 		(mirror y)
@@
 	)
 	(symbol
-		(lib_id "Sensors:CMEJ-0415-42-P")
+		(lib_id "Transducers:CMEJ-0415-42-P")
 		(at 195.58 205.74 0)
 		(mirror y)
@@
 	)
 	(symbol
-		(lib_id "Sensors:CMEJ-0415-42-P")
+		(lib_id "Transducers:CMEJ-0415-42-P")
 		(at 436.88 205.74 0)
 		(mirror y)
@@
 	)
 	(symbol
-		(lib_id "Sensors:CMEJ-0415-42-P")
+		(lib_id "Transducers:CMEJ-0415-42-P")
 		(at 99.06 104.14 0)
 		(mirror y)
@@
 	)
 	(symbol
-		(lib_id "Sensors:CMEJ-0415-42-P")
+		(lib_id "Transducers:CMEJ-0415-42-P")
 		(at 195.58 104.14 0)
 		(mirror y)
@@
 	)
 	(symbol
-		(lib_id "Sensors:CMEJ-0415-42-P")
+		(lib_id "Transducers:CMEJ-0415-42-P")
 		(at 99.06 231.14 0)
 		(mirror y)
@@
 	)
 	(symbol
-		(lib_id "Sensors:CMEJ-0415-42-P")
+		(lib_id "Transducers:CMEJ-0415-42-P")
 		(at 388.62 129.54 0)
 		(mirror y)
@@
 	)
 	(symbol
-		(lib_id "Sensors:CMEJ-0415-42-P")
+		(lib_id "Transducers:CMEJ-0415-42-P")
 		(at 292.1 231.14 0)
 		(mirror y)
@@
 	)
 	(symbol
-		(lib_id "Sensors:CMEJ-0415-42-P")
+		(lib_id "Transducers:CMEJ-0415-42-P")
 		(at 340.36 154.94 0)
 		(mirror y)
@@
 	)
 	(symbol
-		(lib_id "Sensors:CMEJ-0415-42-P")
+		(lib_id "Transducers:CMEJ-0415-42-P")
 		(at 147.32 104.14 0)
 		(mirror y)
@@
 	)
 	(symbol
-		(lib_id "Sensors:CMEJ-0415-42-P")
+		(lib_id "Transducers:CMEJ-0415-42-P")
 		(at 243.84 231.14 0)
 		(mirror y)
@@
 	)
 	(symbol
-		(lib_id "Sensors:CMEJ-0415-42-P")
+		(lib_id "Transducers:CMEJ-0415-42-P")
 		(at 436.88 154.94 0)
 		(mirror y)
@@
 	)
 	(symbol
-		(lib_id "Sensors:CMEJ-0415-42-P")
+		(lib_id "Transducers:CMEJ-0415-42-P")
 		(at 243.84 154.94 0)
 		(mirror y)
@@
 	)
 	(symbol
-		(lib_id "Sensors:CMEJ-0415-42-P")
+		(lib_id "Transducers:CMEJ-0415-42-P")
 		(at 436.88 180.34 0)
 		(mirror y)
@@
 	)
 	(symbol
-		(lib_id "Sensors:CMEJ-0415-42-P")
+		(lib_id "Transducers:CMEJ-0415-42-P")
 		(at 388.62 180.34 0)
 		(mirror y)
@@
 	)
 	(symbol
-		(lib_id "Sensors:CMEJ-0415-42-P")
+		(lib_id "Transducers:CMEJ-0415-42-P")
 		(at 195.58 78.74 0)
 		(mirror y)
@@
 	)
 	(symbol
-		(lib_id "Sensors:CMEJ-0415-42-P")
+		(lib_id "Transducers:CMEJ-0415-42-P")
 		(at 340.36 231.14 0)
 		(mirror y)
@@
 	)
 	(symbol
-		(lib_id "Sensors:CMEJ-0415-42-P")
+		(lib_id "Transducers:CMEJ-0415-42-P")
 		(at 292.1 104.14 0)
 		(mirror y)
@@
 	)
 	(symbol
-		(lib_id "Sensors:CMEJ-0415-42-P")
+		(lib_id "Transducers:CMEJ-0415-42-P")
 		(at 99.06 205.74 0)
 		(mirror y)
@@
 	)
 	(symbol
-		(lib_id "Sensors:CMEJ-0415-42-P")
+		(lib_id "Transducers:CMEJ-0415-42-P")
 		(at 340.36 205.74 0)
 		(mirror y)
@@
 	)
 	(symbol
-		(lib_id "Sensors:CMEJ-0415-42-P")
+		(lib_id "Transducers:CMEJ-0415-42-P")
 		(at 147.32 180.34 0)
 		(mirror y)
@@
 	)
 	(symbol
-		(lib_id "Sensors:CMEJ-0415-42-P")
+		(lib_id "Transducers:CMEJ-0415-42-P")
 		(at 195.58 180.34 0)
 		(mirror y)
@@
 	)
 	(symbol
-		(lib_id "Sensors:CMEJ-0415-42-P")
+		(lib_id "Transducers:CMEJ-0415-42-P")
 		(at 243.84 205.74 0)
 		(mirror y)
@@
 	)
 	(symbol
-		(lib_id "Sensors:CMEJ-0415-42-P")
+		(lib_id "Transducers:CMEJ-0415-42-P")
 		(at 292.1 129.54 0)
 		(mirror y)
@@
 	)
 	(symbol
-		(lib_id "Sensors:CMEJ-0415-42-P")
+		(lib_id "Transducers:CMEJ-0415-42-P")
 		(at 436.88 231.14 0)
 		(mirror y)
@@
 	)
 	(symbol
-		(lib_id "Sensors:CMEJ-0415-42-P")
+		(lib_id "Transducers:CMEJ-0415-42-P")
 		(at 388.62 104.14 0)
 		(mirror y)
@@
 	)
 	(symbol
-		(lib_id "Sensors:CMEJ-0415-42-P")
+		(lib_id "Transducers:CMEJ-0415-42-P")
 		(at 243.84 104.14 0)
 		(mirror y)
@@
 	)
 	(symbol
-		(lib_id "Sensors:CMEJ-0415-42-P")
+		(lib_id "Transducers:CMEJ-0415-42-P")
 		(at 195.58 154.94 0)
 		(mirror y)
@@
 	)
 	(symbol
-		(lib_id "Sensors:CMEJ-0415-42-P")
+		(lib_id "Transducers:CMEJ-0415-42-P")
 		(at 292.1 78.74 0)
 		(mirror y)
@@
 	)
 	(symbol
-		(lib_id "Sensors:CMEJ-0415-42-P")
+		(lib_id "Transducers:CMEJ-0415-42-P")
 		(at 147.32 231.14 0)
 		(mirror y)
@@
 	)
 	(symbol
-		(lib_id "Sensors:CMEJ-0415-42-P")
+		(lib_id "Transducers:CMEJ-0415-42-P")
 		(at 388.62 205.74 0)
 		(mirror y)
@@
 	)
 	(symbol
-		(lib_id "Sensors:CMEJ-0415-42-P")
+		(lib_id "Transducers:CMEJ-0415-42-P")
 		(at 243.84 78.74 0)
 		(mirror y)
@@
 	)
 	(symbol
-		(lib_id "Sensors:CMEJ-0415-42-P")
+		(lib_id "Transducers:CMEJ-0415-42-P")
 		(at 388.62 78.74 0)
 		(mirror y)
@@
 	)
 	(symbol
-		(lib_id "Sensors:CMEJ-0415-42-P")
+		(lib_id "Transducers:CMEJ-0415-42-P")
 		(at 195.58 231.14 0)
 		(mirror y)
@@
 	)
 	(symbol
-		(lib_id "Sensors:CMEJ-0415-42-P")
+		(lib_id "Transducers:CMEJ-0415-42-P")
 		(at 147.32 256.54 0)
 		(mirror y)
@@
 	)
 	(symbol
-		(lib_id "Sensors:CMEJ-0415-42-P")
+		(lib_id "Transducers:CMEJ-0415-42-P")
 		(at 243.84 180.34 0)
 		(mirror y)
@@
 	)
 	(symbol
-		(lib_id "Sensors:CMEJ-0415-42-P")
+		(lib_id "Transducers:CMEJ-0415-42-P")
 		(at 292.1 205.74 0)
 		(mirror y)
@@
 	)
 	(symbol
-		(lib_id "Sensors:CMEJ-0415-42-P")
+		(lib_id "Transducers:CMEJ-0415-42-P")
 		(at 340.36 104.14 0)
 		(mirror y)
@@
 	)
 	(symbol
-		(lib_id "Sensors:CMEJ-0415-42-P")
+		(lib_id "Transducers:CMEJ-0415-42-P")
 		(at 292.1 256.54 0)
 		(mirror y)
@@
 	)
 	(symbol
-		(lib_id "Sensors:CMEJ-0415-42-P")
+		(lib_id "Transducers:CMEJ-0415-42-P")
 		(at 99.06 78.74 0)
 		(mirror y)
@@
 	)
 	(symbol
-		(lib_id "Sensors:CMEJ-0415-42-P")
+		(lib_id "Transducers:CMEJ-0415-42-P")
 		(at 292.1 180.34 0)
 		(mirror y)
@@
 	)
 	(symbol
-		(lib_id "Sensors:CMEJ-0415-42-P")
+		(lib_id "Transducers:CMEJ-0415-42-P")
 		(at 292.1 154.94 0)
 		(mirror y)
@@
 	)
 	(symbol
-		(lib_id "Sensors:CMEJ-0415-42-P")
+		(lib_id "Transducers:CMEJ-0415-42-P")
 		(at 243.84 129.54 0)
 		(mirror y)
@@
 	)
 	(symbol
-		(lib_id "Sensors:CMEJ-0415-42-P")
+		(lib_id "Transducers:CMEJ-0415-42-P")
 		(at 340.36 256.54 0)
 		(mirror y)
@@
 	)
 	(symbol
-		(lib_id "Sensors:CMEJ-0415-42-P")
+		(lib_id "Transducers:CMEJ-0415-42-P")
 		(at 340.36 129.54 0)
 		(mirror y)
@@
 	)
 	(symbol
-		(lib_id "Sensors:CMEJ-0415-42-P")
+		(lib_id "Transducers:CMEJ-0415-42-P")
 		(at 340.36 78.74 0)
 		(mirror y)
@@
 	)
 	(symbol
-		(lib_id "Sensors:CMEJ-0415-42-P")
+		(lib_id "Transducers:CMEJ-0415-42-P")
 		(at 147.32 154.94 0)
 		(mirror y)
