File: KiCAD/ADC.kicad_sch (KiCad schematic)
At the start: 32 parts, among them U2 MAX11059, U3 MAX11059

Commit message: Changed 100pF and 100nF to AVX parts, and gave TPA6211 a pin-1 dot
Parts:
- C10, C20, C21, C22, C23, C24, C25, C27, C28, C29, C30, C31, C32, C33, C34, C35, C36, C37, C38, C9: MPN GCG188R91H104KA01D -> 06035C104KAT2A; Manufacturer Murata -> KYOCERA AVX; SPN 81-GCG188R91H104KA1D -> 581-06035C104KAT2A
Changed lines of the file:
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@@
 			)
 		)
-		(property "Manufacturer" "Murata"
+		(property "Manufacturer" "KYOCERA AVX"
 			(at 76.2 245.745 0)
 			(hide yes)
@@
 			)
 		)
-		(property "MPN" "GCG188R91H104KA01D "
+		(property "MPN" "06035C104KAT2A"
 			(at 76.2 247.65 0)
 			(hide yes)
@@
 			)
 		)
-		(property "SPN" "81-GCG188R91H104KA1D "
+		(property "SPN" "581-06035C104KAT2A"
 			(at 76.2 251.46 0)
 			(hide yes)
@@
 			)
 		)
-		(property "Manufacturer" "Murata"
+		(property "Manufacturer" "KYOCERA AVX"
 			(at 101.6 245.745 0)
 			(hide yes)
@@
 			)
 		)
-		(property "MPN" "GCG188R91H104KA01D "
+		(property "MPN" "06035C104KAT2A"
 			(at 101.6 247.65 0)
 			(hide yes)
@@
 			)
 		)
-		(property "SPN" "81-GCG188R91H104KA1D "
+		(property "SPN" "581-06035C104KAT2A"
 			(at 101.6 251.46 0)
 			(hide yes)
@@
 			)
 		)
-		(property "Manufacturer" "Murata"
+		(property "Manufacturer" "KYOCERA AVX"
 			(at 139.7 245.745 0)
 			(hide yes)
@@
 			)
 		)
-		(property "MPN" "GCG188R91H104KA01D "
+		(property "MPN" "06035C104KAT2A"
 			(at 139.7 247.65 0)
 			(hide yes)
@@
 			)
 		)
-		(property "SPN" "81-GCG188R91H104KA1D "
+		(property "SPN" "581-06035C104KAT2A"
 			(at 139.7 251.46 0)
 			(hide yes)
@@
 			)
 		)
-		(property "Manufacturer" "Murata"
+		(property "Manufacturer" "KYOCERA AVX"
 			(at 101.6 210.185 0)
 			(hide yes)
@@
 			)
 		)
-		(property "MPN" "GCG188R91H104KA01D "
+		(property "MPN" "06035C104KAT2A"
 			(at 101.6 212.09 0)
 			(hide yes)
@@
 			)
 		)
-		(property "SPN" "81-GCG188R91H104KA1D "
+		(property "SPN" "581-06035C104KAT2A"
 			(at 101.6 215.9 0)
 			(hide yes)
@@
 			)
 		)
-		(property "Manufacturer" "Murata"
+		(property "Manufacturer" "KYOCERA AVX"
 			(at 317.5 55.245 0)
 			(hide yes)
@@
 			)
 		)
-		(property "MPN" "GCG188R91H104KA01D "
+		(property "MPN" "06035C104KAT2A"
 			(at 317.5 57.15 0)
 			(hide yes)
@@
 			)
 		)
-		(property "SPN" "81-GCG188R91H104KA1D "
+		(property "SPN" "581-06035C104KAT2A"
 			(at 317.5 60.96 0)
 			(hide yes)
@@
 			)
 		)
-		(property "Manufacturer" "Murata"
+		(property "Manufacturer" "KYOCERA AVX"
 			(at 177.8 245.745 0)
 			(hide yes)
@@
 			)
 		)
-		(property "MPN" "GCG188R91H104KA01D "
+		(property "MPN" "06035C104KAT2A"
 			(at 177.8 247.65 0)
 			(hide yes)
@@
 			)
 		)
-		(property "SPN" "81-GCG188R91H104KA1D "
+		(property "SPN" "581-06035C104KAT2A"
 			(at 177.8 251.46 0)
 			(hide yes)
@@
 			)
 		)
-		(property "Manufacturer" "Murata"
+		(property "Manufacturer" "KYOCERA AVX"
 			(at 190.5 245.745 0)
 			(hide yes)
@@
 			)
 		)
-		(property "MPN" "GCG188R91H104KA01D "
+		(property "MPN" "06035C104KAT2A"
 			(at 190.5 247.65 0)
 			(hide yes)
@@
 			)
 		)
-		(property "SPN" "81-GCG188R91H104KA1D "
+		(property "SPN" "581-06035C104KAT2A"
 			(at 190.5 251.46 0)
 			(hide yes)
@@
 			)
 		)
-		(property "Manufacturer" "Murata"
+		(property "Manufacturer" "KYOCERA AVX"
 			(at 114.3 245.745 0)
 			(hide yes)
@@
 			)
 		)
-		(property "MPN" "GCG188R91H104KA01D "
+		(property "MPN" "06035C104KAT2A"
 			(at 114.3 247.65 0)
 			(hide yes)
@@
 			)
 		)
-		(property "SPN" "81-GCG188R91H104KA1D "
+		(property "SPN" "581-06035C104KAT2A"
 			(at 114.3 251.46 0)
 			(hide yes)
@@
 			)
 		)
-		(property "Manufacturer" "Murata"
+		(property "Manufacturer" "KYOCERA AVX"
 			(at 114.3 210.185 0)
 			(hide yes)
@@
 			)
 		)
-		(property "MPN" "GCG188R91H104KA01D "
+		(property "MPN" "06035C104KAT2A"
 			(at 114.3 212.09 0)
 			(hide yes)
@@
 			)
 		)
-		(property "SPN" "81-GCG188R91H104KA1D "
+		(property "SPN" "581-06035C104KAT2A"
 			(at 114.3 215.9 0)
 			(hide yes)
@@
 			)
 		)
-		(property "Manufacturer" "Murata"
+		(property "Manufacturer" "KYOCERA AVX"
 			(at 88.9 245.745 0)
 			(hide yes)
@@
 			)
 		)
-		(property "MPN" "GCG188R91H104KA01D "
+		(property "MPN" "06035C104KAT2A"
 			(at 88.9 247.65 0)
 			(hide yes)
@@
 			)
 		)
-		(property "SPN" "81-GCG188R91H104KA1D "
+		(property "SPN" "581-06035C104KAT2A"
 			(at 88.9 251.46 0)
 			(hide yes)
@@
 			)
 		)
-		(property "Manufacturer" "Murata"
+		(property "Manufacturer" "KYOCERA AVX"
 			(at 63.5 210.185 0)
 			(hide yes)
@@
 			)
 		)
-		(property "MPN" "GCG188R91H104KA01D "
+		(property "MPN" "06035C104KAT2A"
 			(at 63.5 212.09 0)
 			(hide yes)
@@
 			)
 		)
-		(property "SPN" "81-GCG188R91H104KA1D "
+		(property "SPN" "581-06035C104KAT2A"
 			(at 63.5 215.9 0)
 			(hide yes)
@@
 			)
 		)
-		(property "Manufacturer" "Murata"
+		(property "Manufacturer" "KYOCERA AVX"
 			(at 165.1 245.745 0)
 			(hide yes)
@@
 			)
 		)
-		(property "MPN" "GCG188R91H104KA01D "
+		(property "MPN" "06035C104KAT2A"
 			(at 165.1 247.65 0)
 			(hide yes)
@@
 			)
 		)
-		(property "SPN" "81-GCG188R91H104KA1D "
+		(property "SPN" "581-06035C104KAT2A"
 			(at 165.1 251.46 0)
 			(hide yes)
@@
 			)
 		)
-		(property "Manufacturer" "Murata"
+		(property "Manufacturer" "KYOCERA AVX"
 			(at 88.9 210.185 0)
 			(hide yes)
@@
 			)
 		)
-		(property "MPN" "GCG188R91H104KA01D "
+		(property "MPN" "06035C104KAT2A"
 			(at 88.9 212.09 0)
 			(hide yes)
@@
 			)
 		)
-		(property "SPN" "81-GCG188R91H104KA1D "
+		(property "SPN" "581-06035C104KAT2A"
 			(at 88.9 215.9 0)
 			(hide yes)
@@
 			)
 		)
-		(property "Manufacturer" "Murata"
+		(property "Manufacturer" "KYOCERA AVX"
 			(at 152.4 245.745 0)
 			(hide yes)
@@
 			)
 		)
-		(property "MPN" "GCG188R91H104KA01D "
+		(property "MPN" "06035C104KAT2A"
 			(at 152.4 247.65 0)
 			(hide yes)
@@
 			)
 		)
-		(property "SPN" "81-GCG188R91H104KA1D "
+		(property "SPN" "581-06035C104KAT2A"
 			(at 152.4 251.46 0)
 			(hide yes)
@@
 			)
 		)
-		(property "Manufacturer" "Murata"
+		(property "Manufacturer" "KYOCERA AVX"
 			(at 127 210.185 0)
 			(hide yes)
@@
 			)
 		)
-		(property "MPN" "GCG188R91H104KA01D "
+		(property "MPN" "06035C104KAT2A"
 			(at 127 212.09 0)
 			(hide yes)
@@
 			)
 		)
-		(property "SPN" "81-GCG188R91H104KA1D "
+		(property "SPN" "581-06035C104KAT2A"
 			(at 127 215.9 0)
 			(hide yes)
@@
 			)
 		)
-		(property "Manufacturer" "Murata"
+		(property "Manufacturer" "KYOCERA AVX"
 			(at 76.2 210.185 0)
 			(hide yes)
@@
 			)
 		)
-		(property "MPN" "GCG188R91H104KA01D "
+		(property "MPN" "06035C104KAT2A"
 			(at 76.2 212.09 0)
 			(hide yes)
@@
 			)
 		)
-		(property "SPN" "81-GCG188R91H104KA1D "
+		(property "SPN" "581-06035C104KAT2A"
 			(at 76.2 215.9 0)
 			(hide yes)
@@
 			)
 		)
-		(property "Manufacturer" "Murata"
+		(property "Manufacturer" "KYOCERA AVX"
 			(at 127 245.745 0)
 			(hide yes)
@@
 			)
 		)
-		(property "MPN" "GCG188R91H104KA01D "
+		(property "MPN" "06035C104KAT2A"
 			(at 127 247.65 0)
 			(hide yes)
@@
 			)
 		)
-		(property "SPN" "81-GCG188R91H104KA1D "
+		(property "SPN" "581-06035C104KAT2A"
 			(at 127 251.46 0)
 			(hide yes)
@@
 			)
 		)
-		(property "Manufacturer" "Murata"
+		(property "Manufacturer" "KYOCERA AVX"
 			(at 63.5 245.745 0)
 			(hide yes)
@@
 			)
 		)
-		(property "MPN" "GCG188R91H104KA01D "
+		(property "MPN" "06035C104KAT2A"
 			(at 63.5 247.65 0)
 			(hide yes)
@@
 			)
 		)
-		(property "SPN" "81-GCG188R91H104KA1D "
+		(property "SPN" "581-06035C104KAT2A"
 			(at 63.5 251.46 0)
 			(hide yes)
@@
 			)
 		)
-		(property "Manufacturer" "Murata"
+		(property "Manufacturer" "KYOCERA AVX"
 			(at 139.7 55.245 0)
 			(hide yes)
@@
 			)
 		)
-		(property "MPN" "GCG188R91H104KA01D "
+		(property "MPN" "06035C104KAT2A"
 			(at 139.7 57.15 0)
 			(hide yes)
@@
 			)
 		)
-		(property "SPN" "81-GCG188R91H104KA1D "
+		(property "SPN" "581-06035C104KAT2A"
 			(at 139.7 60.96 0)
 			(hide yes)
@@
 			)
 		)
-		(property "Manufacturer" "Murata"
+		(property "Manufacturer" "KYOCERA AVX"
 			(at 203.2 245.745 0)
 			(hide yes)
@@
 			)
 		)
-		(property "MPN" "GCG188R91H104KA01D "
+		(property "MPN" "06035C104KAT2A"
 			(at 203.2 247.65 0)
 			(hide yes)
@@
 			)
 		)
-		(property "SPN" "81-GCG188R91H104KA1D "
+		(property "SPN" "581-06035C104KAT2A"
 			(at 203.2 251.46 0)
 			(hide yes)
